File: hw-nfc_tag/prj-kicad/cubic-nfc_tag-r01.sch (KiCad schematic (older format))
At the start: 12 parts, among them P1 CONN_1, P2 CONN_1, P3 CONN_1, P4 CONN_1, P5 CONN_1, P6 CONN_1, P7 CONN_1, P8 CONN_1, P9 CONN_1, U1 M24LR04E

Commit message: = UPD: Move ground pad and add a second communication port
Parts:
- removed P7, P8: CONN_1, symbol CONN_1
- added COMM1, COMM2: CONN_3, symbol CONN_3
Connections:
- net labels added: I2C_SCL, I2C_SDA
- wire segments 35 -> 37
- no-connect marks 1 -> 4
Changed lines of the file:
@@
 L GND #PWR02
 U 1 1 5596F544
-P 1850 3700
-F 0 "#PWR02" H 1850 3700 30  0001 C CNN
-F 1 "GND" H 1850 3630 30  0001 C CNN
-F 2 "" H 1850 3700 60  0000 C CNN
-F 3 "" H 1850 3700 60  0000 C CNN
-	1    1850 3700
-	1    0    0    -1
-$EndComp
-Wire Wire Line
-	1850 3700 1850 3600
-Wire Wire Line
-	1850 3600 1750 3600
+P 8150 5300
+F 0 "#PWR02" H 8150 5300 30  0001 C CNN
+F 1 "GND" H 8150 5230 30  0001 C CNN
+F 2 "" H 8150 5300 60  0000 C CNN
+F 3 "" H 8150 5300 60  0000 C CNN
+	1    8150 5300
+	1    0    0    -1
+$EndComp
+Wire Wire Line
+	8150 5300 8150 5200
+Wire Wire Line
+	8150 5200 8050 5200
 $Comp
 L CONN_1 P1
@@
 	1    0    0    -1
 $EndComp
-$Comp
-L CONN_1 P7
-U 1 1 5597011D
-P 4200 3100
-F 0 "P7" H 4280 3100 40  0000 L CNN
-F 1 "CONN_1" H 4200 3155 30  0001 C CNN
-F 2 "" H 4200 3100 60  0000 C CNN
-F 3 "" H 4200 3100 60  0000 C CNN
-	1    4200 3100
-	-1   0    0    1
-$EndComp
-$Comp
-L CONN_1 P8
-U 1 1 55970136
-P 4200 3200
-F 0 "P8" H 4280 3200 40  0000 L CNN
-F 1 "CONN_1" H 4200 3255 30  0001 C CNN
-F 2 "" H 4200 3200 60  0000 C CNN
-F 3 "" H 4200 3200 60  0000 C CNN
-	1    4200 3200
-	-1   0    0    1
-$EndComp
 Wire Wire Line
 	4350 3100 4450 3100
@@
 Wire Wire Line
 	2950 4300 2950 4400
+$Comp
+L CONN_3 COMM1
+U 1 1 55A0D899
+P 7650 5000
+F 0 "COMM1" H 7650 5350 60  0000 C CNN
+F 1 "CONN_3" V 7650 5000 60  0000 C CNN
+F 2 "" H 7650 5000 60  0000 C CNN
+F 3 "" H 7650 5000 60  0000 C CNN
+	1    7650 5000
+	1    0    0    -1
+$EndComp
+Text GLabel 8150 4800 2    50   Output ~ 0
+I2C_SCL
+Text GLabel 4350 3100 0    45   Input ~ 0
+I2C_SCL
+Text GLabel 8150 5000 2    50   BiDi ~ 0
+I2C_SDA
+Wire Wire Line
+	8150 5000 8050 5000
+Wire Wire Line
+	8050 4800 8150 4800
+Text GLabel 4350 3200 0    45   Input ~ 0
+I2C_SDA
+$Comp
+L CONN_3 COMM2
+U 1 1 55A0D94F
+P 10200 5000
+F 0 "COMM2" H 10200 5350 60  0000 C CNN
+F 1 "CONN_3" V 10200 5000 60  0000 C CNN
+F 2 "" H 10200 5000 60  0000 C CNN
+F 3 "" H 10200 5000 60  0000 C CNN
+	1    10200 5000
+	-1   0    0    -1
+$EndComp
+NoConn ~ 9800 4800
+NoConn ~ 9800 5000
+NoConn ~ 9800 5200
 $EndSCHEMATC
